Commit message: updated fork

File: pepper_description/urdf/pepper1.0_generated_urdf/pepperGazebo.xacro (robot description, xacro)
@@ -4,47 +4,47 @@
 	<xacro:property name="PI" value="3.14159265359" />
     <xacro:macro name="DisabledLinks" params="side side_small">
-        <plugin name="${side}Finger11_link" filename="libpepper_gazebo_disable_link_plugin.so">
+        <plugin name="${side}Finger11_link" filename="libroboticsgroup_gazebo_disable_link_plugin.so">
             <link>${side}Finger11_link</link>
         </plugin>
-        <plugin name="${side}Finger12_link" filename="libpepper_gazebo_disable_link_plugin.so">
+        <plugin name="${side}Finger12_link" filename="libroboticsgroup_gazebo_disable_link_plugin.so">
             <link>${side}Finger12_link</link>
         </plugin>
-        <plugin name="${side}Finger13_link" filename="libpepper_gazebo_disable_link_plugin.so">
+        <plugin name="${side}Finger13_link" filename="libroboticsgroup_gazebo_disable_link_plugin.so">
             <link>${side}Finger13_link</link>
         </plugin>
-        <plugin name="${side}Finger21_link" filename="libpepper_gazebo_disable_link_plugin.so">
+        <plugin name="${side}Finger21_link" filename="libroboticsgroup_gazebo_disable_link_plugin.so">
             <link>${side}Finger21_link</link>
         </plugin>
-        <plugin name="${side}Finger22_link" filename="libpepper_gazebo_disable_link_plugin.so">
+        <plugin name="${side}Finger22_link" filename="libroboticsgroup_gazebo_disable_link_plugin.so">
             <link>${side}Finger22_link</link>
         </plugin>
-        <plugin name="${side}Finger23_link" filename="libpepper_gazebo_disable_link_plugin.so">
+        <plugin name="${side}Finger23_link" filename="libroboticsgroup_gazebo_disable_link_plugin.so">
             <link>${side}Finger23_link</link>
         </plugin>
-        <plugin name="${side}Finger31_link" filename="libpepper_gazebo_disable_link_plugin.so">
+        <plugin name="${side}Finger31_link" filename="libroboticsgroup_gazebo_disable_link_plugin.so">
             <link>${side}Finger31_link</link>
         </plugin>
-        <plugin name="${side}Finger32_link" filename="libpepper_gazebo_disable_link_plugin.so">
+        <plugin name="${side}Finger32_link" filename="libroboticsgroup_gazebo_disable_link_plugin.so">
             <link>${side}Finger32_link</link>
         </plugin>
-        <plugin name="${side}Finger33_link" filename="libpepper_gazebo_disable_link_plugin.so">
+        <plugin name="${side}Finger33_link" filename="libroboticsgroup_gazebo_disable_link_plugin.so">
             <link>${side}Finger33_link</link>
         </plugin>
-        <plugin name="${side}Finger41_link" filename="libpepper_gazebo_disable_link_plugin.so">
+        <plugin name="${side}Finger41_link" filename="libroboticsgroup_gazebo_disable_link_plugin.so">
             <link>${side}Finger41_link</link>
         </plugin>
-        <plugin name="${side}Finger42_link" filename="libpepper_gazebo_disable_link_plugin.so">
+        <plugin name="${side}Finger42_link" filename="libroboticsgroup_gazebo_disable_link_plugin.so">
             <link>${side}Finger42_link</link>
         </plugin>
-        <plugin name="${side}Finger43_link" filename="libpepper_gazebo_disable_link_plugin.so">
+        <plugin name="${side}Finger43_link" filename="libroboticsgroup_gazebo_disable_link_plugin.so">
             <link>${side}Finger43_link</link>
         </plugin>
-        <plugin name="${side}Thumb1_link" filename="libpepper_gazebo_disable_link_plugin.so">
+        <plugin name="${side}Thumb1_link" filename="libroboticsgroup_gazebo_disable_link_plugin.so">
             <link>${side}Thumb1_link</link>
         </plugin>
-        <plugin name="${side}Thumb2_link" filename="libpepper_gazebo_disable_link_plugin.so">
+        <plugin name="${side}Thumb2_link" filename="libroboticsgroup_gazebo_disable_link_plugin.so">
             <link>${side}Thumb2_link</link>
         </plugin>
-        <plugin name="${side_small}_gripper" filename="libpepper_gazebo_disable_link_plugin.so">
+        <plugin name="${side_small}_gripper" filename="libroboticsgroup_gazebo_disable_link_plugin.so">
             <link>${side_small}_gripper</link>
         </plugin>
@@ -53,5 +53,5 @@
     <!-- Fingers -->
     <xacro:macro name="FingerMimics" params="side num">
-        <plugin name="mimic_${side}Finger${num}1" filename="libpepper_gazebo_mimic_joint_plugin.so">
+        <plugin name="mimic_${side}Finger${num}1" filename="libroboticsgroup_gazebo_mimic_joint_plugin.so">
             <joint>${side}Hand</joint>
             <mimicJoint>${side}Finger${num}1</mimicJoint>
@@ -59,5 +59,5 @@
             <offset>${PI/4}</offset>
         </plugin>
-        <plugin name="mimic_${side}Finger${num}2" filename="libpepper_gazebo_mimic_joint_plugin.so">
+        <plugin name="mimic_${side}Finger${num}2" filename="libroboticsgroup_gazebo_mimic_joint_plugin.so">
             <joint>${side}Hand</joint>
             <mimicJoint>${side}Finger${num}2</mimicJoint>
@@ -65,5 +65,5 @@
             <offset>${PI/4}</offset>
         </plugin>
-        <plugin name="mimic_${side}Finger${num}3" filename="libpepper_gazebo_mimic_joint_plugin.so">
+        <plugin name="mimic_${side}Finger${num}3" filename="libroboticsgroup_gazebo_mimic_joint_plugin.so">
             <joint>${side}Hand</joint>
             <mimicJoint>${side}Finger${num}3</mimicJoint>
@@ -74,5 +74,5 @@
     <!-- Thumbs -->
     <xacro:macro name="ThumbMimics" params="side">
-        <plugin name="${side}Thumb1" filename="libpepper_gazebo_mimic_joint_plugin.so">
+        <plugin name="${side}Thumb1" filename="libroboticsgroup_gazebo_mimic_joint_plugin.so">
             <joint>${side}Hand</joint>
             <mimicJoint>${side}Thumb1</mimicJoint>
@@ -80,5 +80,5 @@
             <offset>${PI/4}</offset>
         </plugin>
-        <plugin name="${side}Thumb2" filename="libpepper_gazebo_mimic_joint_plugin.so">
+        <plugin name="${side}Thumb2" filename="libroboticsgroup_gazebo_mimic_joint_plugin.so">
             <joint>${side}Hand</joint>
             <mimicJoint>${side}Thumb2</mimicJoint>
@@ -90,5 +90,5 @@
     <gazebo>
         <plugin filename="libgazebo_ros_control.so" name="gazebo_ros_control">
-            <robotNamespace>pepper_dcm</robotNamespace>
+            <robotNamespace></robotNamespace>
             <robotSimType>gazebo_ros_control/DefaultRobotHWSim</robotSimType>
         </plugin>
@@ -314,5 +314,5 @@
     </gazebo>
     <gazebo reference="WheelFL_link">
-        <mu1>0.2</mu1>
+        <mu1>1</mu1>
         <mu2>0</mu2>
         <kp value="10000000.0" />
@@ -323,6 +323,6 @@
     </gazebo>
     <gazebo reference="WheelB_link">
-        <mu1>0.2</mu1>
-        <mu2>0.2</mu2>
+        <mu1>0.5</mu1>
+        <mu2>0.5</mu2>
         <kp value="10000000.0" />
         <kd value="1.0" />
@@ -333,5 +333,5 @@
     <gazebo reference="WheelFR_link">
         <mu1>0</mu1>
-        <mu2>0.2</mu2>
+        <mu2>1</mu2>
         <kp value="10000000.0" />
         <kd value="1.0" />
@@ -691,136 +691,20 @@
   </sensor>
 </gazebo>
-    <!-- Drive controller -->
-    <!--Original drive controller from Aldebaran-->
-<!--<gazebo>
-      <plugin name="differential_drive_controller" filename="libgazebo_ros_diff_drive.so">
-        <alwaysOn>true</alwaysOn>
-        <updateRate>100</updateRate>
-        <robotNamespace>/</robotNamespace>
-        <leftJoint>WheelFL</leftJoint>
-        <rightJoint>WheelFR</rightJoint>
-        <wheelSeparation>0.170</wheelSeparation>
-        <wheelDiameter>0.140</wheelDiameter>
-        <torque>36.9</torque>
-        <commandTopic>cmd_vel</commandTopic>
-        <odometryTopic>odom_diffdrive</odometryTopic>
-        <odometryFrame>odom</odometryFrame>
-        <robotBaseFrame>base_footprint</robotBaseFrame>
-      </plugin>
-    </gazebo>
--->
-    <!-- Custom base plugin Documentation at https://github.com/tu-darmstadt-ros-pkg/hector_gazebo/blob/indigo-devel/hector_gazebo_plugins/src/gazebo_ros_force_based_move.cpp -->
-    <gazebo>
-        <plugin name="base_drive_controller" filename="libpepper_gazebo_ros_force_omni_base.so">
-            <robotNamespace>pepper_robot</robotNamespace>
-            <commandTopic>cmd_vel</commandTopic>
-            <odometryTopic>odom</odometryTopic>
-            <publishOdometryTf>true</publishOdometryTf>
-            <odometryFrame>odom</odometryFrame>
-            <odometryRate>20.0</odometryRate>
-            <robotBaseFrame>Tibia</robotBaseFrame>
-            <yaw_velocity_p_gain>500.0</yaw_velocity_p_gain>
-            <yaw_velocity_i_gain>300.0</yaw_velocity_i_gain>
-            <x_velocity_p_gain>1000.0</x_velocity_p_gain>
-            <x_velocity_i_gain>300.0</x_velocity_i_gain>
-            <y_velocity_p_gain>1000.0</y_velocity_p_gain>
-            <y_velocity_i_gain>300.0</y_velocity_i_gain>
-            <max_torque>8.0</max_torque>
-            <max_force>50.0</max_force>
-        </plugin>
-    </gazebo>
-    <!-- Lasers sensors -->
-    <gazebo reference="SurroundingRightLaser_device_frame">
-      <sensor type="ray" name="laser_sensor_right">
-        <pose>0 0 0 0 0 0</pose>
-        <visualize>false</visualize>
-        <update_rate>10</update_rate>
-        <ray>
-          <scan>
-            <horizontal>
-              <samples>15</samples>
-              <resolution>1</resolution>
-              <min_angle>-0.515</min_angle>
-              <max_angle>0.515</max_angle>
-            </horizontal>
-          </scan>
-          <range>
-            <min>0.10</min>
-            <max>1.5</max>
-            <resolution>0.01</resolution>
-          </range>
-          <noise>
-            <type>gaussian</type>
-            <mean>0.0</mean>
-            <stddev>0.01</stddev>
-          </noise>
-        </ray>
-        <plugin name="gazebo_ros_laser_sensor_right_plugin" filename="libgazebo_ros_laser.so">
-          <topicName>/pepper_robot/laser/right</topicName>
-          <frameName>SurroundingRightLaser_device_frame</frameName>
-        </plugin>
-      </sensor>
-    </gazebo>
-    <gazebo reference="SurroundingLeftLaser_device_frame">
-      <sensor type="ray" name="laser_sensor_left">
-        <pose>0 0 0 0 0 0</pose>
-        <visualize>false</visualize>
-        <update_rate>10</update_rate>
-        <ray>
-          <scan>
-            <horizontal>
-              <samples>15</samples>
-              <resolution>1</resolution>
-              <min_angle>-0.515</min_angle>
-              <max_angle>0.515</max_angle>
-            </horizontal>
-          </scan>
-          <range>
-            <min>0.10</min>
-            <max>1.5</max>
-            <resolution>0.01</resolution>
-          </range>
-          <noise>
-            <type>gaussian</type>
-            <mean>0.0</mean>
-            <stddev>0.01</stddev>
-          </noise>
-        </ray>
-        <plugin name="gazebo_ros_laser_sensor_left_plugin" filename="libgazebo_ros_laser.so">
-          <topicName>/pepper_robot/laser/left</topicName>
-          <frameName>SurroundingLeftLaser_device_frame</frameName>
-        </plugin>
-      </sensor>
-    </gazebo>
-    <gazebo reference="SurroundingFrontLaser_device_frame">
-      <sensor type="ray" name="laser_sensor_front">
-        <pose>0 0 0 0 0 0</pose>
-        <visualize>false</visualize>
-        <update_rate>10</update_rate>
-        <ray>
-          <scan>
-            <horizontal>
-              <samples>15</samples>
-              <resolution>1</resolution>
-              <min_angle>-0.515</min_angle>
-              <max_angle>0.515</max_angle>
-            </horizontal>
-          </scan>
-          <range>
-            <min>0.10</min>
-            <max>1.5</max>
-            <resolution>0.01</resolution>
-          </range>
-          <noise>
-            <type>gaussian</type>
-            <mean>0.0</mean>
-            <stddev>0.01</stddev>
-          </noise>
-        </ray>
-        <plugin name="gazebo_ros_laser_sensor_front_plugin" filename="libgazebo_ros_laser.so">
-          <topicName>/pepper_robot/laser/front</topicName>
-          <frameName>SurroundingFrontLaser_device_frame</frameName>
-        </plugin>
-      </sensor>
-    </gazebo>
+<!-- Drive controller -->
+<gazebo>
+  <plugin name="differential_drive_controller" filename="libgazebo_ros_diff_drive.so">
+    <alwaysOn>true</alwaysOn>
+    <updateRate>100</updateRate>
+    <robotNamespace>/</robotNamespace>
+    <leftJoint>WheelFL</leftJoint>
+    <rightJoint>WheelFR</rightJoint>
+    <wheelSeparation>0.170</wheelSeparation>
+    <wheelDiameter>0.140</wheelDiameter>
+    <torque>36.9</torque>
+    <commandTopic>cmd_vel</commandTopic>
+    <odometryTopic>odom_diffdrive</odometryTopic>
+    <odometryFrame>odom</odometryFrame>
+    <robotBaseFrame>base_footprint</robotBaseFrame>
+  </plugin>
+</gazebo>
 </robot>

File: pepper_description/urdf/pepper1.0_generated_urdf/pepper_fingers.xacro (robot description, xacro)
@@ -4,4 +4,10 @@
  *********************************************************************-->
 <robot name="JulietteY20MP" xmlns:xacro="http://www.ros.org/wiki/xacro">
+   <link name="Lgrasp_frame" />
+	<joint name="Lgrasp_frame_joint" type="fixed">
+		<parent link="l_wrist"/>
+		<child link="Lgrasp_frame"/>
+            <origin rpy="3.1415 0 1.5707" xyz="0.070 0 0"/>
+	</joint>
 	<link name="RFinger41_link">
 		<inertial>
