Commit message: Revert "updated fork" because it killed the simulation and is a big change
This reverts commit 5ae98d9dd78f1ecabb52259522cfe8975dec1bfa.

File: pepper_description/urdf/pepper1.0_generated_urdf/pepperGazebo.xacro (robot description, xacro)
@@ -4,47 +4,47 @@
 	<xacro:property name="PI" value="3.14159265359" />
     <xacro:macro name="DisabledLinks" params="side side_small">
-        <plugin name="${side}Finger11_link" filename="libroboticsgroup_gazebo_disable_link_plugin.so">
+        <plugin name="${side}Finger11_link" filename="libpepper_gazebo_disable_link_plugin.so">
             <link>${side}Finger11_link</link>
         </plugin>
-        <plugin name="${side}Finger12_link" filename="libroboticsgroup_gazebo_disable_link_plugin.so">
+        <plugin name="${side}Finger12_link" filename="libpepper_gazebo_disable_link_plugin.so">
             <link>${side}Finger12_link</link>
         </plugin>
-        <plugin name="${side}Finger13_link" filename="libroboticsgroup_gazebo_disable_link_plugin.so">
+        <plugin name="${side}Finger13_link" filename="libpepper_gazebo_disable_link_plugin.so">
             <link>${side}Finger13_link</link>
         </plugin>
-        <plugin name="${side}Finger21_link" filename="libroboticsgroup_gazebo_disable_link_plugin.so">
+        <plugin name="${side}Finger21_link" filename="libpepper_gazebo_disable_link_plugin.so">
             <link>${side}Finger21_link</link>
         </plugin>
-        <plugin name="${side}Finger22_link" filename="libroboticsgroup_gazebo_disable_link_plugin.so">
+        <plugin name="${side}Finger22_link" filename="libpepper_gazebo_disable_link_plugin.so">
             <link>${side}Finger22_link</link>
         </plugin>
-        <plugin name="${side}Finger23_link" filename="libroboticsgroup_gazebo_disable_link_plugin.so">
+        <plugin name="${side}Finger23_link" filename="libpepper_gazebo_disable_link_plugin.so">
             <link>${side}Finger23_link</link>
         </plugin>
-        <plugin name="${side}Finger31_link" filename="libroboticsgroup_gazebo_disable_link_plugin.so">
+        <plugin name="${side}Finger31_link" filename="libpepper_gazebo_disable_link_plugin.so">
             <link>${side}Finger31_link</link>
         </plugin>
-        <plugin name="${side}Finger32_link" filename="libroboticsgroup_gazebo_disable_link_plugin.so">
+        <plugin name="${side}Finger32_link" filename="libpepper_gazebo_disable_link_plugin.so">
             <link>${side}Finger32_link</link>
         </plugin>
-        <plugin name="${side}Finger33_link" filename="libroboticsgroup_gazebo_disable_link_plugin.so">
+        <plugin name="${side}Finger33_link" filename="libpepper_gazebo_disable_link_plugin.so">
             <link>${side}Finger33_link</link>
         </plugin>
-        <plugin name="${side}Finger41_link" filename="libroboticsgroup_gazebo_disable_link_plugin.so">
+        <plugin name="${side}Finger41_link" filename="libpepper_gazebo_disable_link_plugin.so">
             <link>${side}Finger41_link</link>
         </plugin>
-        <plugin name="${side}Finger42_link" filename="libroboticsgroup_gazebo_disable_link_plugin.so">
+        <plugin name="${side}Finger42_link" filename="libpepper_gazebo_disable_link_plugin.so">
             <link>${side}Finger42_link</link>
         </plugin>
-        <plugin name="${side}Finger43_link" filename="libroboticsgroup_gazebo_disable_link_plugin.so">
+        <plugin name="${side}Finger43_link" filename="libpepper_gazebo_disable_link_plugin.so">
             <link>${side}Finger43_link</link>
         </plugin>
-        <plugin name="${side}Thumb1_link" filename="libroboticsgroup_gazebo_disable_link_plugin.so">
+        <plugin name="${side}Thumb1_link" filename="libpepper_gazebo_disable_link_plugin.so">
             <link>${side}Thumb1_link</link>
         </plugin>
-        <plugin name="${side}Thumb2_link" filename="libroboticsgroup_gazebo_disable_link_plugin.so">
+        <plugin name="${side}Thumb2_link" filename="libpepper_gazebo_disable_link_plugin.so">
             <link>${side}Thumb2_link</link>
         </plugin>
-        <plugin name="${side_small}_gripper" filename="libroboticsgroup_gazebo_disable_link_plugin.so">
+        <plugin name="${side_small}_gripper" filename="libpepper_gazebo_disable_link_plugin.so">
             <link>${side_small}_gripper</link>
         </plugin>
@@ -53,5 +53,5 @@
     <!-- Fingers -->
     <xacro:macro name="FingerMimics" params="side num">
-        <plugin name="mimic_${side}Finger${num}1" filename="libroboticsgroup_gazebo_mimic_joint_plugin.so">
+        <plugin name="mimic_${side}Finger${num}1" filename="libpepper_gazebo_mimic_joint_plugin.so">
             <joint>${side}Hand</joint>
             <mimicJoint>${side}Finger${num}1</mimicJoint>
@@ -59,5 +59,5 @@
             <offset>${PI/4}</offset>
         </plugin>
-        <plugin name="mimic_${side}Finger${num}2" filename="libroboticsgroup_gazebo_mimic_joint_plugin.so">
+        <plugin name="mimic_${side}Finger${num}2" filename="libpepper_gazebo_mimic_joint_plugin.so">
             <joint>${side}Hand</joint>
             <mimicJoint>${side}Finger${num}2</mimicJoint>
@@ -65,5 +65,5 @@
             <offset>${PI/4}</offset>
         </plugin>
-        <plugin name="mimic_${side}Finger${num}3" filename="libroboticsgroup_gazebo_mimic_joint_plugin.so">
+        <plugin name="mimic_${side}Finger${num}3" filename="libpepper_gazebo_mimic_joint_plugin.so">
             <joint>${side}Hand</joint>
             <mimicJoint>${side}Finger${num}3</mimicJoint>
@@ -74,5 +74,5 @@
     <!-- Thumbs -->
     <xacro:macro name="ThumbMimics" params="side">
-        <plugin name="${side}Thumb1" filename="libroboticsgroup_gazebo_mimic_joint_plugin.so">
+        <plugin name="${side}Thumb1" filename="libpepper_gazebo_mimic_joint_plugin.so">
             <joint>${side}Hand</joint>
             <mimicJoint>${side}Thumb1</mimicJoint>
@@ -80,5 +80,5 @@
             <offset>${PI/4}</offset>
         </plugin>
-        <plugin name="${side}Thumb2" filename="libroboticsgroup_gazebo_mimic_joint_plugin.so">
+        <plugin name="${side}Thumb2" filename="libpepper_gazebo_mimic_joint_plugin.so">
             <joint>${side}Hand</joint>
             <mimicJoint>${side}Thumb2</mimicJoint>
@@ -90,5 +90,5 @@
     <gazebo>
         <plugin filename="libgazebo_ros_control.so" name="gazebo_ros_control">
-            <robotNamespace></robotNamespace>
+            <robotNamespace>pepper_dcm</robotNamespace>
             <robotSimType>gazebo_ros_control/DefaultRobotHWSim</robotSimType>
         </plugin>
@@ -314,5 +314,5 @@
     </gazebo>
     <gazebo reference="WheelFL_link">
-        <mu1>1</mu1>
+        <mu1>0.2</mu1>
         <mu2>0</mu2>
         <kp value="10000000.0" />
@@ -323,6 +323,6 @@
     </gazebo>
     <gazebo reference="WheelB_link">
-        <mu1>0.5</mu1>
-        <mu2>0.5</mu2>
+        <mu1>0.2</mu1>
+        <mu2>0.2</mu2>
         <kp value="10000000.0" />
         <kd value="1.0" />
@@ -333,5 +333,5 @@
     <gazebo reference="WheelFR_link">
         <mu1>0</mu1>
-        <mu2>1</mu2>
+        <mu2>0.2</mu2>
         <kp value="10000000.0" />
         <kd value="1.0" />
@@ -691,20 +691,136 @@
   </sensor>
 </gazebo>
-<!-- Drive controller -->
-<gazebo>
-  <plugin name="differential_drive_controller" filename="libgazebo_ros_diff_drive.so">
-    <alwaysOn>true</alwaysOn>
-    <updateRate>100</updateRate>
-    <robotNamespace>/</robotNamespace>
-    <leftJoint>WheelFL</leftJoint>
-    <rightJoint>WheelFR</rightJoint>
-    <wheelSeparation>0.170</wheelSeparation>
-    <wheelDiameter>0.140</wheelDiameter>
-    <torque>36.9</torque>
-    <commandTopic>cmd_vel</commandTopic>
-    <odometryTopic>odom_diffdrive</odometryTopic>
-    <odometryFrame>odom</odometryFrame>
-    <robotBaseFrame>base_footprint</robotBaseFrame>
-  </plugin>
-</gazebo>
+    <!-- Drive controller -->
+    <!--Original drive controller from Aldebaran-->
+<!--<gazebo>
+      <plugin name="differential_drive_controller" filename="libgazebo_ros_diff_drive.so">
+        <alwaysOn>true</alwaysOn>
+        <updateRate>100</updateRate>
+        <robotNamespace>/</robotNamespace>
+        <leftJoint>WheelFL</leftJoint>
+        <rightJoint>WheelFR</rightJoint>
+        <wheelSeparation>0.170</wheelSeparation>
+        <wheelDiameter>0.140</wheelDiameter>
+        <torque>36.9</torque>
+        <commandTopic>cmd_vel</commandTopic>
+        <odometryTopic>odom_diffdrive</odometryTopic>
+        <odometryFrame>odom</odometryFrame>
+        <robotBaseFrame>base_footprint</robotBaseFrame>
+      </plugin>
+    </gazebo>
+-->
+    <!-- Custom base plugin Documentation at https://github.com/tu-darmstadt-ros-pkg/hector_gazebo/blob/indigo-devel/hector_gazebo_plugins/src/gazebo_ros_force_based_move.cpp -->
+    <gazebo>
+        <plugin name="base_drive_controller" filename="libpepper_gazebo_ros_force_omni_base.so">
+            <robotNamespace>pepper_robot</robotNamespace>
+            <commandTopic>cmd_vel</commandTopic>
+            <odometryTopic>odom</odometryTopic>
+            <publishOdometryTf>true</publishOdometryTf>
+            <odometryFrame>odom</odometryFrame>
+            <odometryRate>20.0</odometryRate>
+            <robotBaseFrame>Tibia</robotBaseFrame>
+            <yaw_velocity_p_gain>500.0</yaw_velocity_p_gain>
+            <yaw_velocity_i_gain>300.0</yaw_velocity_i_gain>
+            <x_velocity_p_gain>1000.0</x_velocity_p_gain>
+            <x_velocity_i_gain>300.0</x_velocity_i_gain>
+            <y_velocity_p_gain>1000.0</y_velocity_p_gain>
+            <y_velocity_i_gain>300.0</y_velocity_i_gain>
+            <max_torque>8.0</max_torque>
+            <max_force>50.0</max_force>
+        </plugin>
+    </gazebo>
+    <!-- Lasers sensors -->
+    <gazebo reference="SurroundingRightLaser_device_frame">
+      <sensor type="ray" name="laser_sensor_right">
+        <pose>0 0 0 0 0 0</pose>
+        <visualize>false</visualize>
+        <update_rate>10</update_rate>
+        <ray>
+          <scan>
+            <horizontal>
+              <samples>15</samples>
+              <resolution>1</resolution>
+              <min_angle>-0.515</min_angle>
+              <max_angle>0.515</max_angle>
+            </horizontal>
+          </scan>
+          <range>
+            <min>0.10</min>
+            <max>1.5</max>
+            <resolution>0.01</resolution>
+          </range>
+          <noise>
+            <type>gaussian</type>
+            <mean>0.0</mean>
+            <stddev>0.01</stddev>
+          </noise>
+        </ray>
+        <plugin name="gazebo_ros_laser_sensor_right_plugin" filename="libgazebo_ros_laser.so">
+          <topicName>/pepper_robot/laser/right</topicName>
+          <frameName>SurroundingRightLaser_device_frame</frameName>
+        </plugin>
+      </sensor>
+    </gazebo>
+    <gazebo reference="SurroundingLeftLaser_device_frame">
+      <sensor type="ray" name="laser_sensor_left">
+        <pose>0 0 0 0 0 0</pose>
+        <visualize>false</visualize>
+        <update_rate>10</update_rate>
+        <ray>
+          <scan>
+            <horizontal>
+              <samples>15</samples>
+              <resolution>1</resolution>
+              <min_angle>-0.515</min_angle>
+              <max_angle>0.515</max_angle>
+            </horizontal>
+          </scan>
+          <range>
+            <min>0.10</min>
+            <max>1.5</max>
+            <resolution>0.01</resolution>
+          </range>
+          <noise>
+            <type>gaussian</type>
+            <mean>0.0</mean>
+            <stddev>0.01</stddev>
+          </noise>
+        </ray>
+        <plugin name="gazebo_ros_laser_sensor_left_plugin" filename="libgazebo_ros_laser.so">
+          <topicName>/pepper_robot/laser/left</topicName>
+          <frameName>SurroundingLeftLaser_device_frame</frameName>
+        </plugin>
+      </sensor>
+    </gazebo>
+    <gazebo reference="SurroundingFrontLaser_device_frame">
+      <sensor type="ray" name="laser_sensor_front">
+        <pose>0 0 0 0 0 0</pose>
+        <visualize>false</visualize>
+        <update_rate>10</update_rate>
+        <ray>
+          <scan>
+            <horizontal>
+              <samples>15</samples>
+              <resolution>1</resolution>
+              <min_angle>-0.515</min_angle>
+              <max_angle>0.515</max_angle>
+            </horizontal>
+          </scan>
+          <range>
+            <min>0.10</min>
+            <max>1.5</max>
+            <resolution>0.01</resolution>
+          </range>
+          <noise>
+            <type>gaussian</type>
+            <mean>0.0</mean>
+            <stddev>0.01</stddev>
+          </noise>
+        </ray>
+        <plugin name="gazebo_ros_laser_sensor_front_plugin" filename="libgazebo_ros_laser.so">
+          <topicName>/pepper_robot/laser/front</topicName>
+          <frameName>SurroundingFrontLaser_device_frame</frameName>
+        </plugin>
+      </sensor>
+    </gazebo>
 </robot>

File: pepper_description/urdf/pepper1.0_generated_urdf/pepper_fingers.xacro (robot description, xacro)
@@ -4,10 +4,4 @@
  *********************************************************************-->
 <robot name="JulietteY20MP" xmlns:xacro="http://www.ros.org/wiki/xacro">
-   <link name="Lgrasp_frame" />
-	<joint name="Lgrasp_frame_joint" type="fixed">
-		<parent link="l_wrist"/>
-		<child link="Lgrasp_frame"/>
-            <origin rpy="3.1415 0 1.5707" xyz="0.070 0 0"/>
-	</joint>
 	<link name="RFinger41_link">
 		<inertial>

Commit message: change to namespace from pepper_robot to maqui

File: pepper_description/urdf/pepper1.0_generated_urdf/pepperGazebo.xacro (robot description, xacro)
@@ -3,4 +3,5 @@
     <!-- MACROS FOR DISABLE LINKS -->
 	<xacro:property name="PI" value="3.14159265359" />
+    <xacro:property name="robot_namespace" value="/maqui" />
     <xacro:macro name="DisabledLinks" params="side side_small">
         <plugin name="${side}Finger11_link" filename="libpepper_gazebo_disable_link_plugin.so">
@@ -90,5 +91,5 @@
     <gazebo>
         <plugin filename="libgazebo_ros_control.so" name="gazebo_ros_control">
-            <robotNamespace>pepper_dcm</robotNamespace>
+            <robotNamespace>${robot_namespace}</robotNamespace>
             <robotSimType>gazebo_ros_control/DefaultRobotHWSim</robotSimType>
         </plugin>
@@ -448,5 +449,5 @@
         </camera>
         <plugin name="camera_controller" filename="libgazebo_ros_camera.so">
-            <robotNamespace>/pepper_robot</robotNamespace>
+            <robotNamespace>${robot_namespace}</robotNamespace>
             <alwaysOn>true</alwaysOn>
             <updateRate>5.0</updateRate>
@@ -485,5 +486,5 @@
         </camera>
         <plugin name="camera_controller" filename="libgazebo_ros_camera.so">
-            <robotNamespace>/pepper_robot</robotNamespace>
+            <robotNamespace>${robot_namespace}</robotNamespace>
             <alwaysOn>true</alwaysOn>
             <updateRate>5.0</updateRate>
@@ -520,5 +521,5 @@
           <alwaysOn>true</alwaysOn>
           <updateRate>20.0</updateRate>
-          <cameraName>pepper_robot/camera</cameraName>
+          <cameraName>${robot_namespace}/camera</cameraName>
           <imageTopicName>ir/image_raw</imageTopicName>
           <cameraInfoTopicName>depth/camera_info</cameraInfoTopicName>
@@ -638,5 +639,5 @@
     </ray>
     <plugin filename="libgazebo_ros_range.so" name="gazebo_ros_range">
-      <robotNamespace>/pepper_robot</robotNamespace>
+      <robotNamespace>${robot_namespace}</robotNamespace>
       <gaussianNoise>0.05</gaussianNoise>
       <alwaysOn>true</alwaysOn>
@@ -678,5 +679,5 @@
     </ray>
     <plugin filename="libgazebo_ros_range.so" name="gazebo_ros_range">
-      <robotNamespace>/pepper_robot</robotNamespace>
+      <robotNamespace>${robot_namespace}</robotNamespace>
       <gaussianNoise>0.05</gaussianNoise>
       <alwaysOn>true</alwaysOn>
@@ -713,5 +714,5 @@
     <gazebo>
         <plugin name="base_drive_controller" filename="libpepper_gazebo_ros_force_omni_base.so">
-            <robotNamespace>pepper_robot</robotNamespace>
+            <robotNamespace>${robot_namespace}</robotNamespace>
             <commandTopic>cmd_vel</commandTopic>
             <odometryTopic>odom</odometryTopic>
@@ -757,5 +758,5 @@
         </ray>
         <plugin name="gazebo_ros_laser_sensor_right_plugin" filename="libgazebo_ros_laser.so">
-          <topicName>/pepper_robot/laser/right</topicName>
+          <topicName>${robot_namespace}/laser/right</topicName>
           <frameName>SurroundingRightLaser_device_frame</frameName>
         </plugin>
@@ -788,5 +789,5 @@
         </ray>
         <plugin name="gazebo_ros_laser_sensor_left_plugin" filename="libgazebo_ros_laser.so">
-          <topicName>/pepper_robot/laser/left</topicName>
+          <topicName>${robot_namespace}/laser/left</topicName>
           <frameName>SurroundingLeftLaser_device_frame</frameName>
         </plugin>
@@ -819,5 +820,5 @@
         </ray>
         <plugin name="gazebo_ros_laser_sensor_front_plugin" filename="libgazebo_ros_laser.so">
-          <topicName>/pepper_robot/laser/front</topicName>
+          <topicName>${robot_namespace}/laser/front</topicName>
           <frameName>SurroundingFrontLaser_device_frame</frameName>
         </plugin>

Commit message: modifying pepper laser and collisions of wheels

File: pepper_description/urdf/pepper1.0_generated_urdf/pepperGazebo.xacro (robot description, xacro)
@@ -735,8 +735,8 @@
          the official naoqi ROS driver makes the merge of all the laser and references them to base_footprint frame
     -->
-    <!--<gazebo reference="SurroundingRightLaser_device_frame">
+    <gazebo reference="SurroundingRightLaser_frame">
       <sensor type="ray" name="laser_sensor_right">
         <pose>0 0 0 0 0 0</pose>
-        <visualize>false</visualize>
+        <visualize>true</visualize>
         <update_rate>10</update_rate>
         <ray>
@@ -751,5 +751,5 @@
           <range>
             <min>0.10</min>
-            <max>1.5</max>
+            <max>6.5</max>
             <resolution>0.01</resolution>
           </range>
@@ -762,12 +762,12 @@
         <plugin name="gazebo_ros_laser_sensor_right_plugin" filename="libgazebo_ros_laser.so">
           <topicName>${robot_namespace}/laser/right</topicName>
-          <frameName>SurroundingRightLaser_device_frame</frameName>
+          <frameName>SurroundingRightLaser_frame</frameName>
         </plugin>
       </sensor>
     </gazebo>
-    <gazebo reference="SurroundingLeftLaser_device_frame">
+    <gazebo reference="SurroundingLeftLaser_frame">
       <sensor type="ray" name="laser_sensor_left">
         <pose>0 0 0 0 0 0</pose>
-        <visualize>false</visualize>
+        <visualize>true</visualize>
         <update_rate>10</update_rate>
         <ray>
@@ -782,5 +782,5 @@
           <range>
             <min>0.10</min>
-            <max>1.5</max>
+            <max>6.5</max>
             <resolution>0.01</resolution>
           </range>
@@ -793,12 +793,12 @@
         <plugin name="gazebo_ros_laser_sensor_left_plugin" filename="libgazebo_ros_laser.so">
           <topicName>${robot_namespace}/laser/left</topicName>
-          <frameName>SurroundingLeftLaser_device_frame</frameName>
+          <frameName>SurroundingLeftLaser_frame</frameName>
         </plugin>
       </sensor>
     </gazebo>
-    <gazebo reference="SurroundingFrontLaser_device_frame">
+    <gazebo reference="SurroundingFrontLaser_frame">
       <sensor type="ray" name="laser_sensor_front">
         <pose>0 0 0 0 0 0</pose>
-        <visualize>false</visualize>
+        <visualize>true</visualize>
         <update_rate>10</update_rate>
         <ray>
@@ -813,5 +813,5 @@
           <range>
             <min>0.10</min>
-            <max>1.5</max>
+            <max>6.5</max>
             <resolution>0.01</resolution>
           </range>
@@ -824,9 +824,9 @@
         <plugin name="gazebo_ros_laser_sensor_front_plugin" filename="libgazebo_ros_laser.so">
           <topicName>${robot_namespace}/laser/front</topicName>
-          <frameName>SurroundingFrontLaser_device_frame</frameName>
+          <frameName>SurroundingFrontLaser_frame</frameName>
         </plugin>
       </sensor>
     </gazebo> -->
-    <gazebo reference="base_footprint">
+    <!--gazebo reference="base_footprint">
       <sensor type="ray" name="laser">
         <pose>0 0 0 0 0 0</pose>
@@ -858,4 +858,4 @@
         </plugin>
       </sensor>
-    </gazebo>
+    </gazebo-->
 </robot>

File: pepper_description/urdf/pepper1.0_generated_urdf/pepper_legs.xacro (robot description, xacro)
@@ -43,5 +43,6 @@
 	<link name="Tibia">
 		<inertial>
-			<mass value="11.6015"/>
+			<mass value="11.6015"/> <!--original mass-->
+			<!--mass value="100"/--> <!-- bigger mass to avoid falls-->
 			<inertia ixx="0.129229" ixy="-0.000401943" ixz="0.00048556" iyy="0.122839" iyz="-1.01666e-08" izz="0.108168"/>
 			<origin rpy="0 0 0" xyz="0.00220451 0 -0.185729"/>

File: pepper_description/urdf/pepper1.0_generated_urdf/pepper_visual_collisions.xacro (robot description, xacro)
@@ -111,5 +111,6 @@
 		<collision>
 			<geometry>
-				<mesh filename="package://pepper_meshes/meshes/1.0/WheelFL_0.10.stl" scale="0.1 0.1 0.1"/>
+				<!--mesh filename="package://pepper_meshes/meshes/1.0/WheelFL_0.10.stl" scale="0.1 0.1 0.1"/-->
+				<sphere radius="0.09"/>
 			</geometry>
 			<origin rpy="0 0 0" xyz="0 0 0"/>
@@ -251,5 +252,6 @@
 		<collision>
 			<geometry>
-				<mesh filename="package://pepper_meshes/meshes/1.0/KneePitch_0.10.stl" scale="0.1 0.1 0.1"/>
+				<cylinder length="0.05" radius="0.1"/>
+				<!--mesh filename="package://pepper_meshes/meshes/1.0/KneePitch_0.10.stl" scale="0.1 0.1 0.1"/-->
 			</geometry>
 			<origin rpy="0 0 0" xyz="0 0 0"/>
@@ -461,5 +463,6 @@
 		<collision>
 			<geometry>
-				<mesh filename="package://pepper_meshes/meshes/1.0/WheelB_0.10.stl" scale="0.1 0.1 0.1"/>
+				<!--mesh filename="package://pepper_meshes/meshes/1.0/WheelB_0.10.stl" scale="0.1 0.1 0.1"/-->  <!-- wheels of radius 0.14 meter-->
+				<sphere radius="0.09"/>
 			</geometry>
 			<origin rpy="0 0 0" xyz="0 0 0"/>
@@ -629,5 +632,6 @@
 		<collision>
 			<geometry>
-				<mesh filename="package://pepper_meshes/meshes/1.0/WheelFR_0.10.stl" scale="0.1 0.1 0.1"/>
+				<!--mesh filename="package://pepper_meshes/meshes/1.0/WheelFR_0.10.stl" scale="0.1 0.1 0.1"/-->
+				<sphere radius="0.09"/>
 			</geometry>
 			<origin rpy="0 0 0" xyz="0 0 0"/>
